File: PCB_Designs/AutoThresholdPulseSensor.sch (EAGLE design)
At the start: 52 parts

Commit message: finished first version of board design
Parts:
- removed JP1: (no value), SparkFun-Connectors:M05NO_SILK
- removed LED13, LED27: (no value), SparkFun-LED:LED5MM
- removed U$3: PD-ODD-900-001, Orlando:PD-ODD-900-001
- removed U$4: JST-PTH, Orlando:JST-PTH
- added BREAKOUT: (no value), SparkFun-Connectors:M05NO_SILK
- added C10: 100n, resistor:C-EUC0402
- added JST: JST-PTH, Orlando:JST-PTH
- added LOGO1: OSHW-LOGOS, SparkFun-Aesthetics:OSHW-LOGOS
- added PD1: PD-ODD-900-001, Orlando:PD-ODD-900-001
- added POWER: ON, SparkFun-LED:LED0603
- added R15: 1k, resistor:R-US_R0402
- renumbered U$1 to PD2
Connections:
- new net N$12: POWER.C, R15.1
- net ANODE: no longer LED13.A, LED27.A
- net COMP: now also BREAKOUT.1; no longer JP1.1
- net GND: now also BREAKOUT.4, C10.2, JST.-, PD1.+, R15.2; no longer JP1.4, LED13.C, LED27.C, U$3.+, U$4.-
- net N$1: now also PD1.-; no longer U$3.-
- net PEAK: now also BREAKOUT.2; no longer JP1.2
- net PULSE: now also BREAKOUT.3; no longer JP1.3
- net VCC: now also BREAKOUT.5, C10.1, JST.+, POWER.A; no longer JP1.5, U$4.+
Other:
- note added: "1/2 Vcc Generator"
- note added: "Active Band-pass Filters"
- note added: "Battery and Pwr Indicator"
- note added: "Heartbeat LEDs"
- note added: "Orlando S. Hoilett Calvary Eng, IICEPD Creative Commons License Attribution-NonCommercial-ShareAlike"
- note added: "Pulse Detector"
- note added: "PulseFit V.1.0"
- note added: "Signal Breakout"
- note added: "Threshold Adjuster"
- note added: "Transducer"
- note added: "Transimpedance Amplifier"
- moved on the sheet: C6, C7, C9, GAINP, LED1, LED10, LED11, LED12, LED16, LED22, LED23, LED24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
