File: PCB_Designs/PulseFit-Mini/PulseFit-Mini.sch (EAGLE design)
At the start: 28 parts

Commit message: updated BOM for PulseFit Mini
Other:
- note added: "Orlando S. Hoilett @oshoilett @CalvaryEngineering Made in the @IICEPD Creative Commons License Attribution-NonCommercial- ShareAlike 4.0 Unported"
- note removed: "Heartbeat LEDs"
- note removed: "Orlando S. Hoilett @oshoilett @CalvaryEngineering Made in the @IICEPD Creative Commons License Attribution-NonCommercial- ShareAlike 3.0 Unported"
- moved on the sheet: BREAKOUT, C7, GAINP, LED13, R15
